File: Clock20MHz/Clock20MHz.kicad_sch (KiCad schematic)
At the start: 9 parts, among them J1 OUTPUT, J2 DIVIDER, U1 74AHC04, U2 74HC590A, Y1 20MHz

Commit message: Update to Kicad 6.0
Parts:
- U1: footprint (none) -> Package_DIP:DIP-14_W7.62mm
