File: StepDown_DCDC/StepDown_DCDC.kicad_sch (KiCad schematic)
At the start: 12 parts, among them J1 IN, J2 OUT, U1 LM2596S-5

Commit message: Update
Parts:
- D1: value 1N5822 -> 1N5824; footprint Diode_SMD:D_MELF -> Diode_SMD:D_SMA
Changed lines of the file:
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@@
       (effects (font (size 1.27 1.27)) (justify left))
     )
-    (property "Value" "1N5822" (id 1) (at 116.84 40.3224 90)
+    (property "Value" "1N5824" (id 1) (at 116.84 40.3224 90)
       (effects (font (size 1.27 1.27)) (justify left))
     )
-    (property "Footprint" "Diode_SMD:D_MELF" (id 2) (at 109.855 39.37 0)
+    (property "Footprint" "Diode_SMD:D_SMA" (id 2) (at 109.855 39.37 0)
       (effects (font (size 1.27 1.27)) hide)
     )
@@
     )
     (path "/f8a46177-c207-45e1-aa8c-9ee19c95df87"
-      (reference "D1") (unit 1) (value "1N5822") (footprint "Diode_SMD:D_MELF")
+      (reference "D1") (unit 1) (value "1N5824") (footprint "Diode_SMD:D_SMA")
     )
     (path "/6b388947-0a27-40e1-ac0d-f9ff36a31c7b"

Commit message: Add libraries
Parts:
- removed C3: 15nF, Capacitor_SMD:C_0805_2012Metric, symbol Device:C
- removed R1: 1K, Resistor_SMD:R_0805_2012Metric, symbol Device:R
- removed R2: 3K, Resistor_SMD:R_0805_2012Metric, symbol Device:R
- C1: value 100uF -> 680uF
Connections:
- net +5V: now also U1.4 (FB)
Other:
- moved on the sheet: D2, R3
